File: catch25-servo.kicad_sch (KiCad schematic)
At the start: 1 part

Commit message: update files
Parts:
- added C1, C3, C4: 10u, Capacitor_SMD:C_0603_1608Metric_Pad1.08x0.95mm_HandSolder, symbol Device:C
- added C2: 22u, Capacitor_SMD:C_0603_1608Metric_Pad1.08x0.95mm_HandSolder, symbol Device:C
- added C5: 0.1u, Capacitor_SMD:C_0603_1608Metric_Pad1.08x0.95mm_HandSolder, symbol Device:C
- added D1: 1N4148, Diode_THT:D_DO-35_SOD27_P7.62mm_Horizontal, symbol Diode:1N4148
- added J1, J2: Conn_01x03, Connector_Molex:Molex_SPOX_5268-03A_1x03_P2.50mm_Horizontal, symbol Connector_Generic:Conn_01x03
- added J3: Conn_02x05_Odd_Even, Connector_PinSocket_2.54mm:PinSocket_2x05_P2.54mm_Horizontal, symbol Connector_Generic:Conn_02x05_Odd_Even
- added J4: Conn_01x06, Connector_PinSocket_2.54mm:PinSocket_1x06_P2.54mm_Vertical, symbol Connector_Generic:Conn_01x06
- added J5: Conn_01x02, Connector_AMASS:AMASS_XT30PW-M_1x02_P2.50mm_Horizontal, symbol Connector_Generic:Conn_01x02
- added Q1: 2N3906, Package_TO_SOT_THT:TO-92_Inline, symbol Transistor_BJT:2N3906
- added R2: 1.2k, Resistor_SMD:R_0603_1608Metric_Pad0.98x0.95mm_HandSolder, symbol Device:R
- added R3, R4, R5, R6, R7: 10k, Resistor_SMD:R_0603_1608Metric_Pad0.98x0.95mm_HandSolder, symbol Device:R
- added U1: ~, Package_SO:VSSOP-8_2.3x2mm_P0.5mm, symbol Library:TC7WH241FK
- added U2: MC78L05_SOT89, Package_TO_SOT_SMD:SOT-89-3, symbol Regulator_Linear:MC78L05_SOT89
Connections:
- net GND: now reaches MD1.1 (~{ON}/OFF_CONTROL)
- net GND: now also MD1.3 (1_GROUND), MD1.7 (2_GROUND), C1.2, C2.2, C3.2, C4.2, C5.2, J1.1 (Pin_1), J2.1 (Pin_1), J3.7 (Pin_7), J4.1 (Pin_1), J5.1 (Pin_1), R2.2, R4.1, U1.4 (GND), U2.2 (GND)
- net +BATT: now reaches MD1.2 (VIN)
- net +BATT: now also C2.1, C3.1, D1.1 (K), J5.2 (Pin_2), U2.3 (IN)
- net VCC: now reaches MD1.4 (VOUT)
- net VCC: now also MD1.5 (SENSE), C1.1, J1.2 (Pin_2), J2.2 (Pin_2)
- net at MD1.6 (TRIM): now also R2.1
- new net: Q1.2 (B), R3.2
- new net +5V: C4.1, C5.1, D1.2 (A), J3.1 (Pin_1), Q1.1 (E), R5.2, R6.2, R7.2, U1.8 (VCC), U2.1 (OUT)
- new net SERVO_SIG: J1.3 (Pin_3), J2.3 (Pin_3), R5.1, U1.5 (A2), U1.6 (Y1)
- new net TXEN: Q1.3 (C), R4.2, U1.1 (/G), U1.7 (G)
- new net UART_RX: J3.3 (Pin_3), J4.5 (Pin_5), R7.1, U1.3 (Y2)
- new net UART_TX: J3.5 (Pin_5), J4.4 (Pin_4), R3.1, R6.1, U1.2 (A1)
- no-connect marks 0 -> 14
Other:
- moved on the sheet: MD1

Commit message: update files
Parts:
- added D2: SMAJ45CA, Diode_SMD:D_SMA_Handsoldering, symbol Diode:SMAJ45CA
Connections:
- net +BATT: now also D2.2 (A2)
- net GND: now also D2.1 (A1)
Changed lines of the file:
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@@
 	)
 	(junction
+		(at 121.92 33.02)
+		(diameter 0)
+		(color 0 0 0 0)
+	)
+	(junction
 		(at 35.56 83.82)
 		(diameter 0)
@@
 		(color 0 0 0 0)
 	)
+	(junction
+		(at 121.92 35.56)
+		(diameter 0)
+		(color 0 0 0 0)
+	)
 	(no_connect
 		(at 83.82 137.16)
@@
 	(wire
 		(pts
+			(xy 121.92 35.56) (xy 110.49 35.56)
+		)
+		(stroke
+			(width 0)
+			(type default)
+		)
+	)
+	(wire
+		(pts
 			(xy 233.68 57.15) (xy 233.68 54.61)
 		)
@@
 	(wire
 		(pts
+			(xy 119.38 31.75) (xy 119.38 33.02)
+		)
+		(stroke
+			(width 0)
+			(type default)
+		)
+	)
+	(wire
+		(pts
 			(xy 226.06 64.77) (xy 226.06 62.23)
 		)
@@
 	(wire
 		(pts
+			(xy 110.49 39.37) (xy 106.68 39.37)
+		)
+		(stroke
+			(width 0)
+			(type default)
+		)
+	)
+	(wire
+		(pts
 			(xy 49.53 52.07) (xy 49.53 50.8)
 		)
@@
 	(wire
 		(pts
+			(xy 106.68 31.75) (xy 119.38 31.75)
+		)
+		(stroke
+			(width 0)
+			(type default)
+		)
+	)
+	(wire
+		(pts
 			(xy 66.04 90.17) (xy 81.28 90.17)
 		)
@@
 	(wire
 		(pts
+			(xy 110.49 35.56) (xy 110.49 39.37)
+		)
+		(stroke
+			(width 0)
+			(type default)
+		)
+	)
+	(wire
+		(pts
 			(xy 77.47 92.71) (xy 81.28 92.71)
 		)
@@
 	(wire
 		(pts
+			(xy 119.38 33.02) (xy 121.92 33.02)
+		)
+		(stroke
+			(width 0)
+			(type default)
+		)
+	)
+	(wire
+		(pts
 			(xy 35.56 83.82) (xy 38.1 83.82)
 		)
@@
 					(unit 1)
 				)
+			)
+		)
+	)
+	(symbol
+		(lib_id "Diode:SMAJ45CA")
+		(at 106.68 35.56 90)
+		(unit 1)
+		(exclude_from_sim no)
+		(in_bom yes)
+		(on_board yes)
+		(dnp no)
+		(fields_autoplaced yes)
+		(property "Reference" "D2"
+			(at 109.22 34.2899 90)
+			(effects
+				(font
+					(size 1.27 1.27)
+				)
+				(justify right)
+			)
+		)
+		(property "Value" "SMAJ45CA"
+			(at 109.22 36.8299 90)
+			(effects
+				(font
+					(size 1.27 1.27)
+				)
+				(justify right)
+			)
+		)
+		(property "Footprint" "Diode_SMD:D_SMA_Handsoldering"
+			(at 111.76 35.56 0)
+			(effects
+				(font
+					(size 1.27 1.27)
+				)
+				(hide yes)
+			)
+		)
+		(property "Datasheet" "https://www.littelfuse.com/media?resourcetype=datasheets&itemid=75e32973-b177-4ee3-a0ff-cedaf1abdb93&filename=smaj-datasheet"
+			(at 106.68 35.56 0)
+			(effects
+				(font
+					(size 1.27 1.27)
+				)
+				(hide yes)
+			)
+		)
+		(property "Description" "400W bidirectional Transient Voltage Suppressor, 45.0Vr, SMA(DO-214AC)"
+			(at 106.68 35.56 0)
+			(effects
+				(font
+					(size 1.27 1.27)
+				)
+				(hide yes)
+			)
+		)
+		(pin "1"
+		)
+		(pin "2"
+		)
+		(instances
+			(project ""
+				(path "/258edf5e-88de-4649-9dc2-08e73f17f733"
+					(reference "D2")
+					(unit 1)
+				)

Commit message: update resources
Parts:
- removed U2: MC78L05_SOT89, Package_TO_SOT_SMD:SOT-89-3, symbol Regulator_Linear:MC78L05_SOT89
- added U3: AMS1117-5.0, Package_TO_SOT_SMD:SOT-223-3_TabPin2, symbol Regulator_Linear:AMS1117-5.0
- C2: footprint Capacitor_SMD:C_0603_1608Metric_Pad1.08x0.95mm_HandSolder -> Capacitor_SMD:C_0805_2012Metric_Pad1.18x1.45mm_HandSolder
Connections:
- net +5V: now also U3.2 (VO)
- net +BATT: now also U3.3 (VI)
- net GND: now also U3.1 (GND)
Changed lines of the file:
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@@
 	)
 	(junction
+		(at 41.91 43.18)
+		(diameter 0)
+		(color 0 0 0 0)
+	)
+	(junction
 		(at 238.76 35.56)
 		(diameter 0)
@@
 	)
 	(junction
-		(at 57.15 43.18)
-		(diameter 0)
-		(color 0 0 0 0)
-	)
-	(junction
 		(at 121.92 33.02)
 		(diameter 0)
@@
 	)
 	(junction
-		(at 41.91 43.18)
+		(at 226.06 64.77)
 		(diameter 0)
 		(color 0 0 0 0)
 	)
 	(junction
-		(at 226.06 64.77)
+		(at 57.15 43.18)
 		(diameter 0)
 		(color 0 0 0 0)
@@
 	)
 	(symbol
+		(lib_id "Regulator_Linear:AMS1117-5.0")
+		(at 49.53 43.18 0)
+		(unit 1)
+		(exclude_from_sim no)
+		(in_bom yes)
+		(on_board yes)
+		(dnp no)
+		(fields_autoplaced yes)
+		(property "Reference" "U3"
+			(at 49.53 36.83 0)
+			(effects
+				(font
+					(size 1.27 1.27)
+				)
+			)
+		)
+		(property "Value" "AMS1117-5.0"
+			(at 49.53 39.37 0)
+			(effects
+				(font
+					(size 1.27 1.27)
+				)
+			)
+		)
+		(property "Footprint" "Package_TO_SOT_SMD:SOT-223-3_TabPin2"
+			(at 49.53 38.1 0)
+			(effects
+				(font
+					(size 1.27 1.27)
+				)
+				(hide yes)
+			)
+		)
+		(property "Datasheet" "http://www.advanced-monolithic.com/pdf/ds1117.pdf"
+			(at 52.07 49.53 0)
+			(effects
+				(font
+					(size 1.27 1.27)
+				)
+				(hide yes)
+			)
+		)
+		(property "Description" "1A Low Dropout regulator, positive, 5.0V fixed output, SOT-223"
+			(at 49.53 43.18 0)
+			(effects
+				(font
+					(size 1.27 1.27)
+				)
+				(hide yes)
+			)
+		)
+		(pin "3"
+		)
+		(pin "1"
+		)
+		(pin "2"
+		)
+		(instances
+			(project ""
+				(path "/258edf5e-88de-4649-9dc2-08e73f17f733"
+					(reference "U3")
+					(unit 1)
+				)
+			)
+		)
+	)
+	(symbol
 		(lib_id "Connector_Generic:Conn_01x03")
 		(at 149.86 87.63 0)
@@
 			)
 		)
-		(property "Footprint" "Capacitor_SMD:C_0603_1608Metric_Pad1.08x0.95mm_HandSolder"
+		(property "Footprint" "Capacitor_SMD:C_0805_2012Metric_Pad1.18x1.45mm_HandSolder"
 			(at 147.0152 44.45 0)
 			(effects
@@
 					(unit 1)
 				)
-			)
-		)
-	)
-	(symbol
-		(lib_id "Regulator_Linear:MC78L05_SOT89")
-		(at 49.53 43.18 0)
-		(unit 1)
-		(exclude_from_sim no)
-		(in_bom yes)
-		(on_board yes)
-		(dnp no)
-		(fields_autoplaced yes)
-		(property "Reference" "U2"
-			(at 49.53 36.83 0)
-			(effects
-				(font
-					(size 1.27 1.27)
-				)
-			)
-		)
-		(property "Value" "MC78L05_SOT89"
-			(at 49.53 39.37 0)
-			(effects
-				(font
-					(size 1.27 1.27)
-				)
-			)
-		)
-		(property "Footprint" "Package_TO_SOT_SMD:SOT-89-3"
-			(at 49.53 38.1 0)
-			(effects
-				(font
-					(size 1.27 1.27)
-					(italic yes)
-				)
-				(hide yes)
-			)
-		)
-		(property "Datasheet" "https://www.onsemi.com/pub/Collateral/MC78L00A-D.PDF"
-			(at 49.53 44.45 0)
-			(effects
-				(font
-					(size 1.27 1.27)
-				)
-				(hide yes)
-			)
-		)
-		(property "Description" "Positive 100mA 30V Linear Regulator, Fixed Output 5V, SOT-89"
-			(at 49.53 43.18 0)
-			(effects
-				(font
-					(size 1.27 1.27)
-				)
-				(hide yes)
-			)
-		)
-		(pin "3"
-		)
-		(pin "2"
-		)
-		(pin "1"
-		)
-		(instances
-			(project ""
-				(path "/258edf5e-88de-4649-9dc2-08e73f17f733"
-					(reference "U2")
-					(unit 1)
-				)

Commit message: changed okl to breakout board
Parts:
- removed C1: 10u, Capacitor_SMD:C_0603_1608Metric_Pad1.08x0.95mm_HandSolder, symbol Device:C
- removed C2: 22u, Capacitor_SMD:C_0805_2012Metric_Pad1.18x1.45mm_HandSolder, symbol Device:C
- removed MD1: OKL-T_6-W12N-C, Library:MURATA_OKL-T-6-W12N-C_0, symbol OKL-T_6-W12N-C:OKL-T_6-W12N-C
- removed R2: 1.2k, Resistor_SMD:R_0603_1608Metric_Pad0.98x0.95mm_HandSolder, symbol Device:R
- added U3: ~, Library:OKL, symbol Library:XL4015
- Q1: footprint Package_TO_SOT_THT:TO-92_Inline -> Package_TO_SOT_SMD:SuperSOT-3
- renumbered C3 to C1, C4 to C2, C5 to C3, J3 to J1, J4 to J2, J5 to J3, J1 to J4, J2 to J5, R6 to R1, R3 to R2, R4 to R3, R7 to R4, U3 to U1, U1 to U2
Connections:
- net +BATT: now also U3.1 (IN+)
- net GND: now also U3.2 (IN-), U3.4 (OUT-)
- net VCC: now also U3.3 (OUT+)
- no-connect marks 14 -> 9
